File: daughterboard/rp2040/facade60_daughterboard.kicad_sch (KiCad schematic)
At the start: 13 parts, among them J1 Conn_01x30, J2 USB_C_Receptacle_USB2.0, U1 RT9013-33GB, U5 SRV05-4

Commit message: Replace R1 & R2 to 0402
Parts:
- J1: LCSC (none) -> C2856808; MFR. Part # (none) -> FPC-05F-30PH20
- R10, R9: footprint Resistor_SMD:R_0603_1608Metric -> Resistor_SMD:R_0402_1005Metric
Changed lines of the file:
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@@
       (effects (font (size 1.27 1.27)))
     )
-    (property "Footprint" "Resistor_SMD:R_0603_1608Metric" (at 66.04 42.418 90)
+    (property "Footprint" "Resistor_SMD:R_0402_1005Metric" (at 66.04 42.418 90)
       (effects (font (size 1.27 1.27)) hide)
     )
@@
       (effects (font (size 1.27 1.27)) hide)
     )
-    (property "JLCPCB Part #" "" (at 66.04 40.64 0)
-      (effects (font (size 1.27 1.27)) hide)
-    )
     (property "MFR. Part #" "0402WGF5101TCE" (at 66.04 40.64 0)
       (effects (font (size 1.27 1.27)) hide)
@@
       (effects (font (size 1.27 1.27)))
     )
-    (property "Footprint" "Resistor_SMD:R_0603_1608Metric" (at 66.04 44.958 90)
+    (property "Footprint" "Resistor_SMD:R_0402_1005Metric" (at 66.04 44.958 90)
       (effects (font (size 1.27 1.27)) hide)
     )
     (property "Datasheet" "~" (at 66.04 43.18 0)
-      (effects (font (size 1.27 1.27)) hide)
-    )
-    (property "JLCPCB Part #" "" (at 66.04 43.18 0)
       (effects (font (size 1.27 1.27)) hide)
     )
@@
     )
     (property "Datasheet" "https://www.usb.org/sites/default/files/documents/usb_type-c.zip" (at 45.72 50.8 0)
-      (effects (font (size 1.27 1.27)) hide)
-    )
-    (property "JLCPCB Part #" "" (at 41.91 50.8 0)
       (effects (font (size 1.27 1.27)) hide)
     )
@@
     )
     (property "Datasheet" "~" (at 266.7 119.38 0)
+      (effects (font (size 1.27 1.27)) hide)
+    )
+    (property "LCSC" "C2856808" (at 266.7 119.38 0)
+      (effects (font (size 1.27 1.27)) hide)
+    )
+    (property "MFR. Part #" "FPC-05F-30PH20" (at 266.7 119.38 0)
       (effects (font (size 1.27 1.27)) hide)
     )
@@
       (effects (font (size 1.27 1.27)) hide)
     )
-    (property "JLCPCB Part #" "" (at 71.12 35.56 90)
-      (effects (font (size 1.27 1.27)) hide)
-    )
